File: rgb_chronos.sch (EAGLE design)
At the start: 0 parts

Commit message: LEDs added to dircuit and board
Multiplexing implemented
Parts:
- added U$1, U$10, U$11, U$12, U$13, U$14, U$15, U$16, U$17, U$18, U$19, U$2, U$20, U$21, U$22, U$23, U$24, U$3, U$4, U$5, U$6, U$7, U$8, U$9: LED3_ARGB, pmg-library:LED3_ARGB
Connections:
- new net N$1: U$1.A, U$2.A, U$3.A, U$4.A
- new net N$10: U$12.R, U$16.R, U$20.R, U$24.R, U$4.R, U$8.R
- new net N$11: U$11.G, U$15.G, U$19.G, U$23.G, U$3.G, U$7.G
- new net N$12: U$11.B, U$15.B, U$19.B, U$23.B, U$3.B, U$7.B
- new net N$13: U$10.R, U$14.R, U$18.R, U$2.R, U$22.R, U$6.R
- new net N$14: U$10.G, U$14.G, U$18.G, U$2.G, U$22.G, U$6.G
- new net N$15: U$10.B, U$14.B, U$18.B, U$2.B, U$22.B, U$6.B
- new net N$16: U$1.R, U$13.R, U$17.R, U$21.R, U$5.R, U$9.R
- new net N$17: U$1.G, U$13.G, U$17.G, U$21.G, U$5.G, U$9.G
- new net N$18: U$1.B, U$13.B, U$17.B, U$21.B, U$5.B, U$9.B
- new net N$2: U$21.A, U$22.A, U$23.A, U$24.A
- new net N$3: U$17.A, U$18.A, U$19.A, U$20.A
- new net N$4: U$13.A, U$14.A, U$15.A, U$16.A
- new net N$5: U$10.A, U$11.A, U$12.A, U$9.A
- new net N$6: U$5.A, U$6.A, U$7.A, U$8.A
- new net N$7: U$11.R, U$15.R, U$19.R, U$23.R, U$3.R, U$7.R
- new net N$8: U$12.B, U$16.B, U$20.B, U$24.B, U$4.B, U$8.B
- new net N$9: U$12.G, U$16.G, U$20.G, U$24.G, U$4.G, U$8.G

Commit message: Display nets renamed
Connections:
- net N$1 renamed COL0
- net N$10 renamed ROW3_R
- net N$11 renamed ROW2_G
- net N$12 renamed ROW2_B
- net N$13 renamed ROW1_R
- net N$14 renamed ROW1_G
- net N$15 renamed ROW1_B
- net N$16 renamed ROW0_R
- net N$17 renamed ROW0_G
- net N$18 renamed ROW0_B
- net N$2 renamed COL5
- net N$3 renamed COL4
- net N$4 renamed COL3
- net N$5 renamed COL2
- net N$6 renamed COL1
- net N$7 renamed ROW2_R
- net N$8 renamed ROW3_B
- net N$9 renamed ROW3_G
Changed lines of the file:
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@@
 </busses>
 <nets>
-<net name="N$1" class="0">
+<net name="COL0" class="0">
 <segment>
 <pinref part="U$1" gate="G$1" pin="A"/>
@@
 </segment>
 </net>
-<net name="N$2" class="0">
+<net name="COL5" class="0">
 <segment>
 <pinref part="U$21" gate="G$1" pin="A"/>
@@
 </segment>
 </net>
-<net name="N$3" class="0">
+<net name="COL4" class="0">
 <segment>
 <pinref part="U$17" gate="G$1" pin="A"/>
@@
 </segment>
 </net>
-<net name="N$4" class="0">
+<net name="COL3" class="0">
 <segment>
 <pinref part="U$13" gate="G$1" pin="A"/>
@@
 </segment>
 </net>
-<net name="N$5" class="0">
+<net name="COL2" class="0">
 <segment>
 <pinref part="U$9" gate="G$1" pin="A"/>
@@
 </segment>
 </net>
-<net name="N$6" class="0">
+<net name="COL1" class="0">
 <segment>
 <pinref part="U$5" gate="G$1" pin="A"/>
@@
 </segment>
 </net>
-<net name="N$7" class="0">
+<net name="ROW2_R" class="0">
 <segment>
 <pinref part="U$3" gate="G$1" pin="R"/>
@@
 </segment>
 </net>
-<net name="N$8" class="0">
+<net name="ROW3_B" class="0">
 <segment>
 <pinref part="U$4" gate="G$1" pin="B"/>
@@
 </segment>
 </net>
-<net name="N$9" class="0">
+<net name="ROW3_G" class="0">
 <segment>
 <wire x1="-203.2" y1="96.52" x2="-160.02" y2="96.52" width="0.1524" layer="91"/>
@@
 </segment>
 </net>
-<net name="N$10" class="0">
+<net name="ROW3_R" class="0">
 <segment>
 <pinref part="U$4" gate="G$1" pin="R"/>
@@
 </segment>
 </net>
-<net name="N$11" class="0">
+<net name="ROW2_G" class="0">
 <segment>
 <pinref part="U$3" gate="G$1" pin="G"/>
@@
 </segment>
 </net>
-<net name="N$12" class="0">
+<net name="ROW2_B" class="0">
 <segment>
 <pinref part="U$3" gate="G$1" pin="B"/>
@@
 </segment>
 </net>
-<net name="N$13" class="0">
+<net name="ROW1_R" class="0">
 <segment>
 <pinref part="U$2" gate="G$1" pin="R"/>
@@
 </segment>
 </net>
-<net name="N$14" class="0">
+<net name="ROW1_G" class="0">
 <segment>
 <pinref part="U$2" gate="G$1" pin="G"/>
@@
 </segment>
 </net>
-<net name="N$15" class="0">
+<net name="ROW1_B" class="0">
 <segment>
 <pinref part="U$2" gate="G$1" pin="B"/>
@@
 </segment>
 </net>
-<net name="N$16" class="0">
+<net name="ROW0_R" class="0">
 <segment>
 <pinref part="U$1" gate="G$1" pin="R"/>
@@
 </segment>
 </net>
-<net name="N$17" class="0">
+<net name="ROW0_G" class="0">
 <segment>
 <pinref part="U$1" gate="G$1" pin="G"/>
@@
 </segment>
 </net>
-<net name="N$18" class="0">
+<net name="ROW0_B" class="0">
 <segment>
 <pinref part="U$1" gate="G$1" pin="B"/>

Commit message: Added LED part number
Parts:
- U$1, U$10, U$11, U$12, U$13, U$14, U$15, U$16, U$17, U$18, U$19, U$2, U$20, U$21, U$22, U$23, U$24, U$3, U$4, U$5, U$6, U$7, U$8, U$9: value LED3_ARGB -> ASMB-MTB0-0A3A2
Changed lines of the file:
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@@
 </classes>
 <parts>
-<part name="U$1" library="pmg-library" deviceset="LED3_ARGB" device=""/>
-<part name="U$2" library="pmg-library" deviceset="LED3_ARGB" device=""/>
-<part name="U$3" library="pmg-library" deviceset="LED3_ARGB" device=""/>
-<part name="U$4" library="pmg-library" deviceset="LED3_ARGB" device=""/>
-<part name="U$5" library="pmg-library" deviceset="LED3_ARGB" device=""/>
-<part name="U$6" library="pmg-library" deviceset="LED3_ARGB" device=""/>
-<part name="U$7" library="pmg-library" deviceset="LED3_ARGB" device=""/>
-<part name="U$8" library="pmg-library" deviceset="LED3_ARGB" device=""/>
-<part name="U$9" library="pmg-library" deviceset="LED3_ARGB" device=""/>
-<part name="U$10" library="pmg-library" deviceset="LED3_ARGB" device=""/>
-<part name="U$11" library="pmg-library" deviceset="LED3_ARGB" device=""/>
-<part name="U$12" library="pmg-library" deviceset="LED3_ARGB" device=""/>
-<part name="U$13" library="pmg-library" deviceset="LED3_ARGB" device=""/>
-<part name="U$14" library="pmg-library" deviceset="LED3_ARGB" device=""/>
-<part name="U$15" library="pmg-library" deviceset="LED3_ARGB" device=""/>
-<part name="U$16" library="pmg-library" deviceset="LED3_ARGB" device=""/>
-<part name="U$17" library="pmg-library" deviceset="LED3_ARGB" device=""/>
-<part name="U$18" library="pmg-library" deviceset="LED3_ARGB" device=""/>
-<part name="U$19" library="pmg-library" deviceset="LED3_ARGB" device=""/>
-<part name="U$20" library="pmg-library" deviceset="LED3_ARGB" device=""/>
-<part name="U$21" library="pmg-library" deviceset="LED3_ARGB" device=""/>
-<part name="U$22" library="pmg-library" deviceset="LED3_ARGB" device=""/>
-<part name="U$23" library="pmg-library" deviceset="LED3_ARGB" device=""/>
-<part name="U$24" library="pmg-library" deviceset="LED3_ARGB" device=""/>
+<part name="U$1" library="pmg-library" deviceset="LED3_ARGB" device="" value="ASMB-MTB0-0A3A2"/>
+<part name="U$2" library="pmg-library" deviceset="LED3_ARGB" device="" value="ASMB-MTB0-0A3A2"/>
+<part name="U$3" library="pmg-library" deviceset="LED3_ARGB" device="" value="ASMB-MTB0-0A3A2"/>
+<part name="U$4" library="pmg-library" deviceset="LED3_ARGB" device="" value="ASMB-MTB0-0A3A2"/>
+<part name="U$5" library="pmg-library" deviceset="LED3_ARGB" device="" value="ASMB-MTB0-0A3A2"/>
+<part name="U$6" library="pmg-library" deviceset="LED3_ARGB" device="" value="ASMB-MTB0-0A3A2"/>
+<part name="U$7" library="pmg-library" deviceset="LED3_ARGB" device="" value="ASMB-MTB0-0A3A2"/>
+<part name="U$8" library="pmg-library" deviceset="LED3_ARGB" device="" value="ASMB-MTB0-0A3A2"/>
+<part name="U$9" library="pmg-library" deviceset="LED3_ARGB" device="" value="ASMB-MTB0-0A3A2"/>
+<part name="U$10" library="pmg-library" deviceset="LED3_ARGB" device="" value="ASMB-MTB0-0A3A2"/>
+<part name="U$11" library="pmg-library" deviceset="LED3_ARGB" device="" value="ASMB-MTB0-0A3A2"/>
+<part name="U$12" library="pmg-library" deviceset="LED3_ARGB" device="" value="ASMB-MTB0-0A3A2"/>
+<part name="U$13" library="pmg-library" deviceset="LED3_ARGB" device="" value="ASMB-MTB0-0A3A2"/>
+<part name="U$14" library="pmg-library" deviceset="LED3_ARGB" device="" value="ASMB-MTB0-0A3A2"/>
+<part name="U$15" library="pmg-library" deviceset="LED3_ARGB" device="" value="ASMB-MTB0-0A3A2"/>
+<part name="U$16" library="pmg-library" deviceset="LED3_ARGB" device="" value="ASMB-MTB0-0A3A2"/>
+<part name="U$17" library="pmg-library" deviceset="LED3_ARGB" device="" value="ASMB-MTB0-0A3A2"/>
+<part name="U$18" library="pmg-library" deviceset="LED3_ARGB" device="" value="ASMB-MTB0-0A3A2"/>
+<part name="U$19" library="pmg-library" deviceset="LED3_ARGB" device="" value="ASMB-MTB0-0A3A2"/>
+<part name="U$20" library="pmg-library" deviceset="LED3_ARGB" device="" value="ASMB-MTB0-0A3A2"/>
+<part name="U$21" library="pmg-library" deviceset="LED3_ARGB" device="" value="ASMB-MTB0-0A3A2"/>
+<part name="U$22" library="pmg-library" deviceset="LED3_ARGB" device="" value="ASMB-MTB0-0A3A2"/>
+<part name="U$23" library="pmg-library" deviceset="LED3_ARGB" device="" value="ASMB-MTB0-0A3A2"/>
+<part name="U$24" library="pmg-library" deviceset="LED3_ARGB" device="" value="ASMB-MTB0-0A3A2"/>
 </parts>
 <sheets>
